File: mini-v1.14-macrofab-rtg_SS_1.sch (KiCad schematic (older format))
At the start: 25 parts, among them U2 TLV70233PDBVR

Commit message: footprints assigned
Parts:
- C1, C10, C11, C12, C13, C2: footprint RCL_C0603 -> mini-v1.14-macrofab-rtg:RCL_C0603
- D1: footprint MF_DISCRETE_SEMICONDUCTOR_SOD-123 -> mini-v1.14-macrofab-rtg:MF_DISCRETE_SEMICONDUCTOR_SOD-123
- J1: footprint MF_CONNECTORS_MICROUSB-RIGHT -> mini-v1.14-macrofab-rtg:MF_CONNECTORS_MICROUSB-RIGHT
- L1: footprint LMDPARTS_C0603 -> mini-v1.14-macrofab-rtg:LMDPARTS_C0603
- LED1, LED2, LED3, LED4: footprint ADAFRUIT_CHIP-LED0603 -> mini-v1.14-macrofab-rtg:ADAFRUIT_CHIP-LED0603
- R2, R20, R21, R26, R3, R35, R4: footprint MF_PASSIVES_R0603 -> mini-v1.14-macrofab-rtg:MF_PASSIVES_R0603
- U$1: footprint LMDPARTS_LQFP48 -> mini-v1.14-macrofab-rtg:LMDPARTS_LQFP48
- U$10, U$13: footprint LMDPARTS_SOD123 -> mini-v1.14-macrofab-rtg:LMDPARTS_SOD123
- U$12: footprint LMDPARTS_SC70-6 -> mini-v1.14-macrofab-rtg:LMDPARTS_SC70-6
- U2: footprint MF_IC_POWER_SOT-23-5 -> mini-v1.14-macrofab-rtg:MF_IC_POWER_SOT-23-5
Changed lines of the file:
@@
 F 0 "C1" H 6490 10674 70  0000 L BNN
 F 1 "1uF" H 6489 10485 70  0000 L BNN
-F 2 "RCL_C0603" H 6440 10440 65  0001 L TNN
+F 2 "mini-v1.14-macrofab-rtg:RCL_C0603" H 6440 10440 65  0001 L TNN
 F 3 "" H 6450 10650 60  0001 C CNN
 	1    6450 10650
@@
 F 0 "C2" H 8490 10775 70  0000 L BNN
 F 1 "1uF" H 8490 10585 70  0000 L BNN
-F 2 "RCL_C0603" H 8440 10540 65  0001 L TNN
+F 2 "mini-v1.14-macrofab-rtg:RCL_C0603" H 8440 10540 65  0001 L TNN
 F 3 "" H 8450 10750 60  0001 C CNN
 	1    8450 10750
@@
 F 0 "C10" H 10090 4574 70  0000 L BNN
 F 1 "0.1uF" H 10089 4385 70  0000 L BNN
-F 2 "RCL_C0603" H 10040 4340 65  0001 L TNN
+F 2 "mini-v1.14-macrofab-rtg:RCL_C0603" H 10040 4340 65  0001 L TNN
 F 3 "" H 10050 4550 60  0001 C CNN
 	1    10050 4550
@@
 F 0 "C11" H 11090 6274 70  0000 L BNN
 F 1 "0.1uF" H 11089 6085 70  0000 L BNN
-F 2 "RCL_C0603" H 11040 6040 65  0001 L TNN
+F 2 "mini-v1.14-macrofab-rtg:RCL_C0603" H 11040 6040 65  0001 L TNN
 F 3 "" H 11050 6250 60  0001 C CNN
 	1    11050 6250
@@
 F 0 "C12" H 6490 4374 70  0000 L BNN
 F 1 "0.1uF" H 6489 4185 70  0000 L BNN
-F 2 "RCL_C0603" H 6440 4140 65  0001 L TNN
+F 2 "mini-v1.14-macrofab-rtg:RCL_C0603" H 6440 4140 65  0001 L TNN
 F 3 "" H 6450 4350 60  0001 C CNN
 	1    6450 4350
@@
 F 0 "C13" H 6690 7374 70  0000 L BNN
 F 1 "0.1uF" H 6689 7185 70  0000 L BNN
-F 2 "RCL_C0603" H 6640 7140 65  0001 L TNN
+F 2 "mini-v1.14-macrofab-rtg:RCL_C0603" H 6640 7140 65  0001 L TNN
 F 3 "" H 6650 7350 60  0001 C CNN
 	1    6650 7350
@@
 F 0 "D1" H 5950 10350 40  0000 L BNN
 F 1 "BAT42" H 5950 10151 40  0000 L BNN
-F 2 "MF_DISCRETE_SEMICONDUCTOR_SOD-123" H 6140 10040 65  0001 L TNN
+F 2 "mini-v1.14-macrofab-rtg:MF_DISCRETE_SEMICONDUCTOR_SOD-123" H 6140 10040 65  0001 L TNN
 F 3 "" H 6150 10250 60  0001 C CNN
 	1    6150 10250
@@
 F 0 "J1" H 6650 9650 40  0000 L BNN
 F 1 "~" H 6840 9040 65  0001 L TNN
-F 2 "MF_CONNECTORS_MICROUSB-RIGHT" H 6840 8940 65  0001 L TNN
+F 2 "mini-v1.14-macrofab-rtg:MF_CONNECTORS_MICROUSB-RIGHT" H 6840 8940 65  0001 L TNN
 F 3 "" H 6850 9150 60  0001 C CNN
 	1    6850 9150
@@
 F 0 "L1" V 5900 8550 70  0000 L BNN
 F 1 "ferrite" V 6100 8550 70  0000 L BNN
-F 2 "LMDPARTS_C0603" H 5940 8540 65  0001 L TNN
+F 2 "mini-v1.14-macrofab-rtg:LMDPARTS_C0603" H 5940 8540 65  0001 L TNN
 F 3 "" H 5950 8750 60  0001 C CNN
 	1    5950 8750
@@
 F 0 "LED1" V 9790 7570 70  0000 L BNN
 F 1 "~" H 9640 7640 65  0001 L TNN
-F 2 "ADAFRUIT_CHIP-LED0603" H 9640 7540 65  0001 L TNN
+F 2 "mini-v1.14-macrofab-rtg:ADAFRUIT_CHIP-LED0603" H 9640 7540 65  0001 L TNN
 F 3 "" H 9650 7750 60  0001 C CNN
 	1    9650 7750
@@
 F 0 "LED2" V 9490 7570 70  0000 L BNN
 F 1 "~" H 9340 7640 65  0001 L TNN
-F 2 "ADAFRUIT_CHIP-LED0603" H 9340 7540 65  0001 L TNN
+F 2 "mini-v1.14-macrofab-rtg:ADAFRUIT_CHIP-LED0603" H 9340 7540 65  0001 L TNN
 F 3 "" H 9350 7750 60  0001 C CNN
 	1    9350 7750
@@
 F 0 "LED3" V 10090 7570 70  0000 L BNN
 F 1 "~" H 9940 7640 65  0001 L TNN
-F 2 "ADAFRUIT_CHIP-LED0603" H 9940 7540 65  0001 L TNN
+F 2 "mini-v1.14-macrofab-rtg:ADAFRUIT_CHIP-LED0603" H 9940 7540 65  0001 L TNN
 F 3 "" H 9950 7750 60  0001 C CNN
 	1    9950 7750
@@
 F 0 "LED4" V 10390 7570 70  0000 L BNN
 F 1 "~" H 10240 7640 65  0001 L TNN
-F 2 "ADAFRUIT_CHIP-LED0603" H 10240 7540 65  0001 L TNN
+F 2 "mini-v1.14-macrofab-rtg:ADAFRUIT_CHIP-LED0603" H 10240 7540 65  0001 L TNN
 F 3 "" H 10250 7750 60  0001 C CNN
 	1    10250 7750
@@
 F 0 "R2" H 9150 7450 40  0000 L BNN
 F 1 "2k" H 9350 7450 40  0000 L BNN
-F 2 "MF_PASSIVES_R0603" H 9340 7140 65  0001 L TNN
+F 2 "mini-v1.14-macrofab-rtg:MF_PASSIVES_R0603" H 9340 7140 65  0001 L TNN
 F 3 "" H 9350 7350 60  0001 C CNN
 	1    9350 7350
@@
 F 0 "R3" H 9450 7450 40  0000 L BNN
 F 1 "2k" H 9650 7450 40  0000 L BNN
-F 2 "MF_PASSIVES_R0603" H 9640 7140 65  0001 L TNN
+F 2 "mini-v1.14-macrofab-rtg:MF_PASSIVES_R0603" H 9640 7140 65  0001 L TNN
 F 3 "" H 9650 7350 60  0001 C CNN
 	1    9650 7350
@@
 F 0 "R4" H 5750 9550 40  0000 L BNN
 F 1 "100k" H 5950 9550 40  0000 L BNN
-F 2 "MF_PASSIVES_R0603" H 5940 9240 65  0001 L TNN
+F 2 "mini-v1.14-macrofab-rtg:MF_PASSIVES_R0603" H 5940 9240 65  0001 L TNN
 F 3 "" H 5950 9450 60  0001 C CNN
 	1    5950 9450
@@
 F 0 "R20" H 9750 7450 40  0000 L BNN
 F 1 "2k" H 9950 7450 40  0000 L BNN
-F 2 "MF_PASSIVES_R0603" H 9940 7140 65  0001 L TNN
+F 2 "mini-v1.14-macrofab-rtg:MF_PASSIVES_R0603" H 9940 7140 65  0001 L TNN
 F 3 "" H 9950 7350 60  0001 C CNN
 	1    9950 7350
@@
 F 0 "R21" H 10050 7450 40  0000 L BNN
 F 1 "2k" H 10250 7450 40  0000 L BNN
-F 2 "MF_PASSIVES_R0603" H 10240 7140 65  0001 L TNN
+F 2 "mini-v1.14-macrofab-rtg:MF_PASSIVES_R0603" H 10240 7140 65  0001 L TNN
 F 3 "" H 10250 7350 60  0001 C CNN
 	1    10250 7350
@@
 F 0 "R26" H 6750 8750 40  0000 L BNN
 F 1 "604k" H 6950 8750 40  0000 L BNN
-F 2 "MF_PASSIVES_R0603" H 6940 8440 65  0001 L TNN
+F 2 "mini-v1.14-macrofab-rtg:MF_PASSIVES_R0603" H 6940 8440 65  0001 L TNN
 F 3 "" H 6950 8650 60  0001 C CNN
 	1    6950 8650
@@
 F 0 "R35" H 6650 10950 40  0000 L BNN
 F 1 "825k" H 6850 10950 40  0000 L BNN
-F 2 "MF_PASSIVES_R0603" H 6840 10640 65  0001 L TNN
+F 2 "mini-v1.14-macrofab-rtg:MF_PASSIVES_R0603" H 6840 10640 65  0001 L TNN
 F 3 "" H 6850 10850 60  0001 C CNN
 	1    6850 10850
@@
 F 0 "U$1" H 7850 4250 70  0000 L BNN
 F 1 "STM32F042C6T6-LQFP48" H 7851 6950 70  0000 L BNN
-F 2 "LMDPARTS_LQFP48" H 8340 5540 65  0001 L TNN
+F 2 "mini-v1.14-macrofab-rtg:LMDPARTS_LQFP48" H 8340 5540 65  0001 L TNN
 F 3 "" H 8350 5750 60  0001 C CNN
 	1    8350 5750
@@
 F 0 "U$10" H 13750 6170 50  0000 L BNN
 F 1 "SMF6.0A" H 13750 5870 50  0000 L BNN
-F 2 "LMDPARTS_SOD123" H 13940 5840 65  0001 L TNN
+F 2 "mini-v1.14-macrofab-rtg:LMDPARTS_SOD123" H 13940 5840 65  0001 L TNN
 F 3 "" H 13950 6050 60  0001 C CNN
 	1    13950 6050
@@
 F 0 "U$12" H 7651 9750 70  0000 L BNN
 F 1 "SP3002-04JTG" H 7650 9050 70  0000 L BNN
-F 2 "LMDPARTS_SC70-6" H 7840 9040 65  0001 L TNN
+F 2 "mini-v1.14-macrofab-rtg:LMDPARTS_SC70-6" H 7840 9040 65  0001 L TNN
 F 3 "" H 7850 9250 60  0001 C CNN
 	1    7850 9250
@@
 F 0 "U$13" H 8750 9170 50  0000 L BNN
 F 1 "SMF6.0A" H 8750 8870 50  0000 L BNN
-F 2 "LMDPARTS_SOD123" H 8940 8840 65  0001 L TNN
+F 2 "mini-v1.14-macrofab-rtg:LMDPARTS_SOD123" H 8940 8840 65  0001 L TNN
 F 3 "" H 8950 9050 60  0001 C CNN
 	1    8950 9050
@@
 F 0 "U2" H 7250 10550 40  0000 L BNN
 F 1 "TLV70233PDBVR" H 7250 10450 40  0000 L BNN
-F 2 "MF_IC_POWER_SOT-23-5" H 7240 10140 65  0001 L TNN
+F 2 "mini-v1.14-macrofab-rtg:MF_IC_POWER_SOT-23-5" H 7240 10140 65  0001 L TNN
 F 3 "" H 7250 10350 60  0001 C CNN
 	1    7250 10350
