File: mini-v1.14-macrofab-rtg_SS_2.sch (KiCad schematic (older format))
At the start: 40 parts

Commit message: footprints assigned
Parts:
- C19, C20, C4, C5, C6, C7: footprint MF_PASSIVES_C0603 -> mini-v1.14-macrofab-rtg:MF_PASSIVES_C0603
- JP3: footprint PINHEAD_2X03 -> mini-v1.14-macrofab-rtg:PINHEAD_2X03
- R10, R11, R12, R22, R23, R24, R27, R28, R29, R30, R31, R32, R33, R34, R36, R37, R39, R40, R41, R5, R6, R8, R9: footprint MF_PASSIVES_R0603 -> mini-v1.14-macrofab-rtg:MF_PASSIVES_R0603
- TP3, TP4, TP5, TP6: footprint TESTPAD_B1_27 -> mini-v1.14-macrofab-rtg:TESTPAD_B1_27
- U$15, U$16, U$17, U$7: footprint LMDPARTS_SOT23-5 -> mini-v1.14-macrofab-rtg:LMDPARTS_SOT23-5
- U$2, U$4: footprint LMDPARTS_SC70-6 -> mini-v1.14-macrofab-rtg:LMDPARTS_SC70-6
