File: mini-v1.14-macrofab-rtg_SS_3.sch (KiCad schematic (older format))
At the start: 29 parts, among them U1 BSS138, U3 BSS138

Commit message: footprints assigned
Parts:
- C14, C16, C17, C18, C8, C9: footprint MF_PASSIVES_C0603 -> mini-v1.14-macrofab-rtg:MF_PASSIVES_C0603
- C15: footprint RCL_C0603 -> mini-v1.14-macrofab-rtg:RCL_C0603
- C3: footprint MF_PASSIVES_CP4MM -> mini-v1.14-macrofab-rtg:MF_PASSIVES_CP4MM
- LASER71, TP2: footprint TESTPAD_B2_54 -> mini-v1.14-macrofab-rtg:TESTPAD_B2_54
- LD1: footprint MINI-V1.14-MACROFAB-RTG_SCOTT_LASERDIODE3 -> mini-v1.14-macrofab-rtg:MINI-V1.14-MACROFAB-RTG_SCOTT_LASERDIODE3
- R13, R14, R15, R16, R17, R18, R19, R25, R38, R42, R43, R7: footprint MF_PASSIVES_R0603 -> mini-v1.14-macrofab-rtg:MF_PASSIVES_R0603
- U$14: footprint LMDPARTS_SDR0403 -> mini-v1.14-macrofab-rtg:LMDPARTS_SDR0403
- U$5, U$8: footprint LMDPARTS_SOT23-5 -> mini-v1.14-macrofab-rtg:LMDPARTS_SOT23-5
- U$9: footprint LMDPARTS_SOD123 -> mini-v1.14-macrofab-rtg:LMDPARTS_SOD123
- U1, U3: footprint MF_DISCRETE_SEMICONDUCTOR_SOT-23-3 -> mini-v1.14-macrofab-rtg:MF_DISCRETE_SEMICONDUCTOR_SOT-23-3
Changed lines of the file:
@@
 F 0 "C3" H 9350 5950 40  0000 L BNN
 F 1 "10uF" H 9350 5750 40  0000 L BNN
-F 2 "MF_PASSIVES_CP4MM" H 9240 5640 65  0001 L TNN
+F 2 "mini-v1.14-macrofab-rtg:MF_PASSIVES_CP4MM" H 9240 5640 65  0001 L TNN
 F 3 "" H 9250 5850 60  0001 C CNN
 	1    9250 5850
@@
 F 0 "C8" H 10150 8150 40  0000 L BNN
 F 1 "0.1uF" H 10150 7950 40  0000 L BNN
-F 2 "MF_PASSIVES_C0603" H 10040 7840 65  0001 L TNN
+F 2 "mini-v1.14-macrofab-rtg:MF_PASSIVES_C0603" H 10040 7840 65  0001 L TNN
 F 3 "" H 10050 8050 60  0001 C CNN
 	1    10050 8050
@@
 F 0 "C9" H 6250 5850 40  0000 L BNN
 F 1 "1uF" H 6250 5650 40  0000 L BNN
-F 2 "MF_PASSIVES_C0603" H 6140 5540 65  0001 L TNN
+F 2 "mini-v1.14-macrofab-rtg:MF_PASSIVES_C0603" H 6140 5540 65  0001 L TNN
 F 3 "" H 6150 5750 60  0001 C CNN
 	1    6150 5750
@@
 F 0 "C14" H 10350 8150 40  0000 L BNN
 F 1 "0.1uF" H 10350 7950 40  0000 L BNN
-F 2 "MF_PASSIVES_C0603" H 10240 7840 65  0001 L TNN
+F 2 "mini-v1.14-macrofab-rtg:MF_PASSIVES_C0603" H 10240 7840 65  0001 L TNN
 F 3 "" H 10250 8050 60  0001 C CNN
 	1    10250 8050
@@
 F 0 "C15" V 9025 5390 70  0000 L BNN
 F 1 "560pF/50V" V 8675 5650 70  0000 R TNN
-F 2 "RCL_C0603" H 8840 5340 65  0001 L TNN
+F 2 "mini-v1.14-macrofab-rtg:RCL_C0603" H 8840 5340 65  0001 L TNN
 F 3 "" H 8850 5550 60  0001 C CNN
 	1    8850 5550
@@
 F 0 "C16" H 11750 9250 40  0000 L BNN
 F 1 "0.1uF" H 11750 9050 40  0000 L BNN
-F 2 "MF_PASSIVES_C0603" H 11640 8940 65  0001 L TNN
+F 2 "mini-v1.14-macrofab-rtg:MF_PASSIVES_C0603" H 11640 8940 65  0001 L TNN
 F 3 "" H 11650 9150 60  0001 C CNN
 	1    11650 9150
@@
 F 0 "C17" H 6550 5850 40  0000 L BNN
 F 1 "1uF" H 6550 5650 40  0000 L BNN
-F 2 "MF_PASSIVES_C0603" H 6440 5540 65  0001 L TNN
+F 2 "mini-v1.14-macrofab-rtg:MF_PASSIVES_C0603" H 6440 5540 65  0001 L TNN
 F 3 "" H 6450 5750 60  0001 C CNN
 	1    6450 5750
@@
 F 0 "C18" H 6850 5850 40  0000 L BNN
 F 1 "0.1uF" H 6850 5650 40  0000 L BNN
-F 2 "MF_PASSIVES_C0603" H 6740 5540 65  0001 L TNN
+F 2 "mini-v1.14-macrofab-rtg:MF_PASSIVES_C0603" H 6740 5540 65  0001 L TNN
 F 3 "" H 6750 5750 60  0001 C CNN
 	1    6750 5750
@@
 F 0 "LASER71" H 12400 8000 70  0000 L BNN
 F 1 "TPB2,54" H 12440 7840 65  0001 L TNN
-F 2 "TESTPAD_B2_54" H 12440 7740 65  0001 L TNN
+F 2 "mini-v1.14-macrofab-rtg:TESTPAD_B2_54" H 12440 7740 65  0001 L TNN
 F 3 "" H 12450 7950 60  0001 C CNN
 	1    12450 7950
@@
 F 0 "LD1" V 12390 6670 70  0000 L BNN
 F 1 "SCOTT_LASERDIODELD3" H 12240 6740 65  0001 L TNN
-F 2 "MINI-V1.14-MACROFAB-RTG_SCOTT_LASERDIODE3" H 12240 6640 65  0001 L TNN
+F 2 "mini-v1.14-macrofab-rtg:MINI-V1.14-MACROFAB-RTG_SCOTT_LASERDIODE3" H 12240 6640 65  0001 L TNN
 F 3 "" H 12250 6850 60  0001 C CNN
 	1    12250 6850
@@
 F 0 "R7" H 9050 7449 40  0000 L BNN
 F 1 "2k" H 9250 7450 40  0000 L BNN
-F 2 "MF_PASSIVES_R0603" H 9240 7140 65  0001 L TNN
+F 2 "mini-v1.14-macrofab-rtg:MF_PASSIVES_R0603" H 9240 7140 65  0001 L TNN
 F 3 "" H 9250 7350 60  0001 C CNN
 	1    9250 7350
@@
 F 0 "R13" H 8550 7849 40  0000 L BNN
 F 1 "1k69" H 8750 7850 40  0000 L BNN
-F 2 "MF_PASSIVES_R0603" H 8740 7540 65  0001 L TNN
+F 2 "mini-v1.14-macrofab-rtg:MF_PASSIVES_R0603" H 8740 7540 65  0001 L TNN
 F 3 "" H 8750 7750 60  0001 C CNN
 	1    8750 7750
@@
 F 0 "R14" H 9050 7849 40  0000 L BNN
 F 1 "1k69" H 9250 7850 40  0000 L BNN
-F 2 "MF_PASSIVES_R0603" H 9240 7540 65  0001 L TNN
+F 2 "mini-v1.14-macrofab-rtg:MF_PASSIVES_R0603" H 9240 7540 65  0001 L TNN
 F 3 "" H 9250 7750 60  0001 C CNN
 	1    9250 7750
@@
 F 0 "R15" H 9450 8149 40  0000 L BNN
 F 1 "1k69" H 9650 8150 40  0000 L BNN
-F 2 "MF_PASSIVES_R0603" H 9640 7840 65  0001 L TNN
+F 2 "mini-v1.14-macrofab-rtg:MF_PASSIVES_R0603" H 9640 7840 65  0001 L TNN
 F 3 "" H 9650 8050 60  0001 C CNN
 	1    9650 8050
@@
 F 0 "R16" H 11150 7750 40  0000 L BNN
 F 1 "10" H 11350 7750 40  0000 L BNN
-F 2 "MF_PASSIVES_R0603" H 11340 7440 65  0001 L TNN
+F 2 "mini-v1.14-macrofab-rtg:MF_PASSIVES_R0603" H 11340 7440 65  0001 L TNN
 F 3 "" H 11350 7650 60  0001 C CNN
 	1    11350 7650
@@
 F 0 "R17" H 8750 5250 40  0000 L BNN
 F 1 "63k4" H 8950 5250 40  0000 L BNN
-F 2 "MF_PASSIVES_R0603" H 8940 4940 65  0001 L TNN
+F 2 "mini-v1.14-macrofab-rtg:MF_PASSIVES_R0603" H 8940 4940 65  0001 L TNN
 F 3 "" H 8950 5150 60  0001 C CNN
 	1    8950 5150
@@
 F 0 "R18" H 8450 5950 40  0000 L BNN
 F 1 "13k3" H 8650 5950 40  0000 L BNN
-F 2 "MF_PASSIVES_R0603" H 8640 5640 65  0001 L TNN
+F 2 "mini-v1.14-macrofab-rtg:MF_PASSIVES_R0603" H 8640 5640 65  0001 L TNN
 F 3 "" H 8650 5850 60  0001 C CNN
 	1    8650 5850
@@
 F 0 "R19" H 6950 5650 40  0000 L BNN
 F 1 "825k" H 7150 5650 40  0000 L BNN
-F 2 "MF_PASSIVES_R0603" H 7140 5340 65  0001 L TNN
+F 2 "mini-v1.14-macrofab-rtg:MF_PASSIVES_R0603" H 7140 5340 65  0001 L TNN
 F 3 "" H 7150 5550 60  0001 C CNN
 	1    7150 5550
@@
 F 0 "R25" H 12050 8350 40  0000 L BNN
 F 1 "10" H 12250 8350 40  0000 L BNN
-F 2 "MF_PASSIVES_R0603" H 12240 8040 65  0001 L TNN
+F 2 "mini-v1.14-macrofab-rtg:MF_PASSIVES_R0603" H 12240 8040 65  0001 L TNN
 F 3 "" H 12250 8250 60  0001 C CNN
 	1    12250 8250
@@
 F 0 "R38" H 12450 8350 40  0000 L BNN
 F 1 "1k69" H 12650 8350 40  0000 L BNN
-F 2 "MF_PASSIVES_R0603" H 12640 8040 65  0001 L TNN
+F 2 "mini-v1.14-macrofab-rtg:MF_PASSIVES_R0603" H 12640 8040 65  0001 L TNN
 F 3 "" H 12650 8250 60  0001 C CNN
 	1    12650 8250
@@
 F 0 "R42" H 12250 8850 40  0000 L BNN
 F 1 "N/C" H 12450 8850 40  0000 L BNN
-F 2 "MF_PASSIVES_R0603" H 12440 8540 65  0001 L TNN
+F 2 "mini-v1.14-macrofab-rtg:MF_PASSIVES_R0603" H 12440 8540 65  0001 L TNN
 F 3 "" H 12450 8750 60  0001 C CNN
 	1    12450 8750
@@
 F 0 "R43" H 11150 8949 40  0000 L BNN
 F 1 "1k69" H 11350 8950 40  0000 L BNN
-F 2 "MF_PASSIVES_R0603" H 11340 8640 65  0001 L TNN
+F 2 "mini-v1.14-macrofab-rtg:MF_PASSIVES_R0603" H 11340 8640 65  0001 L TNN
 F 3 "" H 11350 8850 60  0001 C CNN
 	1    11350 8850
@@
 F 0 "TP2" H 12700 9100 70  0000 L BNN
 F 1 "GND" H 12740 8940 65  0001 L TNN
-F 2 "TESTPAD_B2_54" H 12740 8840 65  0001 L TNN
+F 2 "mini-v1.14-macrofab-rtg:TESTPAD_B2_54" H 12740 8840 65  0001 L TNN
 F 3 "" H 12750 9050 60  0001 C CNN
 	1    12750 9050
@@
 F 0 "U$5" H 10350 8070 50  0000 L BNN
 F 1 "LMC7101" H 10350 7581 50  0000 L BNN
-F 2 "LMDPARTS_SOT23-5" H 10640 7540 65  0001 L TNN
+F 2 "mini-v1.14-macrofab-rtg:LMDPARTS_SOT23-5" H 10640 7540 65  0001 L TNN
 F 3 "" H 10650 7750 60  0001 C CNN
 	1    10650 7750
@@
 F 0 "U$8" H 7550 5950 70  0000 L BNN
 F 1 "LMR62014" H 7940 5440 65  0001 L TNN
-F 2 "LMDPARTS_SOT23-5" H 7940 5340 65  0001 L TNN
+F 2 "mini-v1.14-macrofab-rtg:LMDPARTS_SOT23-5" H 7940 5340 65  0001 L TNN
 F 3 "" H 7950 5550 60  0001 C CNN
 	1    7950 5550
@@
 F 0 "U$9" H 8650 4870 50  0000 L BNN
 F 1 "MBR0520" H 8650 4570 50  0000 L BNN
-F 2 "LMDPARTS_SOD123" H 8840 4540 65  0001 L TNN
+F 2 "mini-v1.14-macrofab-rtg:LMDPARTS_SOD123" H 8840 4540 65  0001 L TNN
 F 3 "" H 8850 4750 60  0001 C CNN
 	1    8850 4750
@@
 F 0 "U$14" V 7950 5090 86  0000 R TNN
 F 1 "SDR0403-100ML" V 7750 5390 86  0000 R TNN
-F 2 "LMDPARTS_SDR0403" H 7840 4740 65  0001 L TNN
+F 2 "mini-v1.14-macrofab-rtg:LMDPARTS_SDR0403" H 7840 4740 65  0001 L TNN
 F 3 "" H 7850 4950 60  0001 C CNN
 	1    7850 4950
@@
 F 0 "U1" H 12150 7850 40  0000 L BNN
 F 1 "BSS138" H 12150 7450 40  0000 R TNN
-F 2 "MF_DISCRETE_SEMICONDUCTOR_SOT-23-3" H 12140 7440 65  0001 L TNN
+F 2 "mini-v1.14-macrofab-rtg:MF_DISCRETE_SEMICONDUCTOR_SOT-23-3" H 12140 7440 65  0001 L TNN
 F 3 "" H 12150 7650 60  0001 C CNN
 	1    12150 7650
@@
 F 0 "U3" H 12150 9050 40  0000 L BNN
 F 1 "BSS138" H 12150 8650 40  0000 R TNN
-F 2 "MF_DISCRETE_SEMICONDUCTOR_SOT-23-3" H 12140 8640 65  0001 L TNN
+F 2 "mini-v1.14-macrofab-rtg:MF_DISCRETE_SEMICONDUCTOR_SOT-23-3" H 12140 8640 65  0001 L TNN
 F 3 "" H 12150 8850 60  0001 C CNN
 	1    12150 8850
