File: mini-v1.14-macrofab-rtg_SS_4.sch (KiCad schematic (older format))
At the start: 10 parts

Commit message: footprints assigned
Parts:
- 3V71, GND71, NRST71, SWCLK71, SWDIO71, VUSB71: footprint TESTPAD_B1_27 -> mini-v1.14-macrofab-rtg:TESTPAD_B1_27
- JP4: footprint PINHEAD_1X02 -> mini-v1.14-macrofab-rtg:PINHEAD_1X02
- JP5, JP6: footprint PINHEAD_2X03 -> mini-v1.14-macrofab-rtg:PINHEAD_2X03
- R1: footprint MF_PASSIVES_R0603 -> mini-v1.14-macrofab-rtg:MF_PASSIVES_R0603
Changed lines of the file:
@@
 F 0 "3V71" H 13800 6000 70  0000 L BNN
 F 1 "TPB1,27" H 13840 5840 65  0001 L TNN
-F 2 "TESTPAD_B1_27" H 13840 5740 65  0001 L TNN
+F 2 "mini-v1.14-macrofab-rtg:TESTPAD_B1_27" H 13840 5740 65  0001 L TNN
 F 3 "" H 13850 5950 60  0001 C CNN
 	1    13850 5950
@@
 F 0 "GND71" H 14100 6600 70  0000 L BNN
 F 1 "TPB1,27" H 14140 6440 65  0001 L TNN
-F 2 "TESTPAD_B1_27" H 14140 6340 65  0001 L TNN
+F 2 "mini-v1.14-macrofab-rtg:TESTPAD_B1_27" H 14140 6340 65  0001 L TNN
 F 3 "" H 14150 6550 60  0001 C CNN
 	1    14150 6550
@@
 F 0 "JP4" H 11100 5775 70  0000 L BNN
 F 1 "~" H 11340 5440 65  0001 L TNN
-F 2 "PINHEAD_1X02" H 11340 5340 65  0001 L TNN
+F 2 "mini-v1.14-macrofab-rtg:PINHEAD_1X02" H 11340 5340 65  0001 L TNN
 F 3 "" H 11350 5550 60  0001 C CNN
 	1    11350 5550
@@
 F 0 "JP5" H 9500 8975 70  0000 L BNN
 F 1 "~" H 9740 8640 65  0001 L TNN
-F 2 "PINHEAD_2X03" H 9740 8540 65  0001 L TNN
+F 2 "mini-v1.14-macrofab-rtg:PINHEAD_2X03" H 9740 8540 65  0001 L TNN
 F 3 "" H 9750 8750 60  0001 C CNN
 	1    9750 8750
@@
 F 0 "JP6" H 10800 8975 70  0000 L BNN
 F 1 "~" H 11040 8640 65  0001 L TNN
-F 2 "PINHEAD_2X03" H 11040 8540 65  0001 L TNN
+F 2 "mini-v1.14-macrofab-rtg:PINHEAD_2X03" H 11040 8540 65  0001 L TNN
 F 3 "" H 11050 8750 60  0001 C CNN
 	1    11050 8750
@@
 F 0 "NRST71" H 14100 6300 70  0000 L BNN
 F 1 "TPB1,27" H 14140 6140 65  0001 L TNN
-F 2 "TESTPAD_B1_27" H 14140 6040 65  0001 L TNN
+F 2 "mini-v1.14-macrofab-rtg:TESTPAD_B1_27" H 14140 6040 65  0001 L TNN
 F 3 "" H 14150 6250 60  0001 C CNN
 	1    14150 6250
@@
 F 0 "R1" H 10750 5950 40  0000 L BNN
 F 1 "13k3" H 10950 5950 40  0000 L BNN
-F 2 "MF_PASSIVES_R0603" H 10940 5640 65  0001 L TNN
+F 2 "mini-v1.14-macrofab-rtg:MF_PASSIVES_R0603" H 10940 5640 65  0001 L TNN
 F 3 "" H 10950 5850 60  0001 C CNN
 	1    10950 5850
@@
 F 0 "SWCLK71" H 13800 6300 70  0000 L BNN
 F 1 "TPB1,27" H 13840 6140 65  0001 L TNN
-F 2 "TESTPAD_B1_27" H 13840 6040 65  0001 L TNN
+F 2 "mini-v1.14-macrofab-rtg:TESTPAD_B1_27" H 13840 6040 65  0001 L TNN
 F 3 "" H 13850 6250 60  0001 C CNN
 	1    13850 6250
@@
 F 0 "SWDIO71" H 13800 6600 70  0000 L BNN
 F 1 "TPB1,27" H 13840 6440 65  0001 L TNN
-F 2 "TESTPAD_B1_27" H 13840 6340 65  0001 L TNN
+F 2 "mini-v1.14-macrofab-rtg:TESTPAD_B1_27" H 13840 6340 65  0001 L TNN
 F 3 "" H 13850 6550 60  0001 C CNN
 	1    13850 6550
@@
 F 0 "VUSB71" H 14100 6000 70  0000 L BNN
 F 1 "TPB1,27" H 14140 5840 65  0001 L TNN
-F 2 "TESTPAD_B1_27" H 14140 5740 65  0001 L TNN
+F 2 "mini-v1.14-macrofab-rtg:TESTPAD_B1_27" H 14140 5740 65  0001 L TNN
 F 3 "" H 14150 5950 60  0001 C CNN
 	1    14150 5950
