File: mini-v1.14-macrofab-rtg.kicad_pcb (KiCad board)
At the start: 2 copper layers, 38 x 66 mm, 106 parts, among them U1 BSS138, U2 TLV70233PDBVR, U3 BSS138

Commit message: Netlist generated and applied
Parts:
- J1, JP3, JP4, JP5, JP6, LED1, LED2, LED3, LED4: value (none) -> ~
Connections:
- net 2V2 renamed /mini-v1.14-macrofab-rtg_SS_2/2V2
- net COARSE1 renamed /mini-v1.14-macrofab-rtg_SS_2/COARSE1
- net FINE1 renamed /mini-v1.14-macrofab-rtg_SS_2/FINE1
- net FINE3 renamed /mini-v1.14-macrofab-rtg_SS_2/FINE3
- net N$1 renamed /mini-v1.14-macrofab-rtg_SS_3/N$1
- net N$10 renamed /mini-v1.14-macrofab-rtg_SS_2/N$10
- net N$11 renamed /mini-v1.14-macrofab-rtg_SS_3/N$11
- net N$12 renamed /mini-v1.14-macrofab-rtg_SS_1/N$12
- net N$13 renamed /mini-v1.14-macrofab-rtg_SS_1/N$13
- net N$14 renamed /mini-v1.14-macrofab-rtg_SS_1/N$14
- net N$16 renamed /mini-v1.14-macrofab-rtg_SS_3/N$16
- net N$17 renamed /mini-v1.14-macrofab-rtg_SS_3/N$17
- net N$18 renamed SLD
- net N$19 renamed /mini-v1.14-macrofab-rtg_SS_3/N$19
- net N$2 renamed /mini-v1.14-macrofab-rtg_SS_1/N$2
- net N$20 renamed /mini-v1.14-macrofab-rtg_SS_3/N$20
- net N$21 renamed /mini-v1.14-macrofab-rtg_SS_3/N$21
- net N$22 renamed /mini-v1.14-macrofab-rtg_SS_2/N$22
- net N$24 renamed /mini-v1.14-macrofab-rtg_SS_1/N$24
- net N$25 renamed /mini-v1.14-macrofab-rtg_SS_3/N$25
- net N$26 renamed /mini-v1.14-macrofab-rtg_SS_3/N$26
- net N$27 renamed /mini-v1.14-macrofab-rtg_SS_1/N$27
- net N$28 renamed /mini-v1.14-macrofab-rtg_SS_1/N$28
- net N$29 renamed /mini-v1.14-macrofab-rtg_SS_1/N$29
- net N$3 renamed /mini-v1.14-macrofab-rtg_SS_1/N$3
- net N$30 renamed /mini-v1.14-macrofab-rtg_SS_2/N$30
- net N$31 renamed /mini-v1.14-macrofab-rtg_SS_2/N$31
- net N$32 renamed /mini-v1.14-macrofab-rtg_SS_2/N$32
- net N$35 renamed /mini-v1.14-macrofab-rtg_SS_2/N$35
- net N$36 renamed /mini-v1.14-macrofab-rtg_SS_2/N$36
- net N$5 renamed /mini-v1.14-macrofab-rtg_SS_1/N$5
- net N$6 renamed /mini-v1.14-macrofab-rtg_SS_3/N$6
- net N$7 renamed /mini-v1.14-macrofab-rtg_SS_2/N$7
- net N$8 renamed /mini-v1.14-macrofab-rtg_SS_2/N$8
- net N$9 renamed /mini-v1.14-macrofab-rtg_SS_3/N$9
- net OUT renamed /mini-v1.14-macrofab-rtg_SS_2/OUT
- net OUT1 renamed /mini-v1.14-macrofab-rtg_SS_2/OUT1
- net OUT2 renamed /mini-v1.14-macrofab-rtg_SS_2/OUT2
- net OUT3 renamed /mini-v1.14-macrofab-rtg_SS_2/OUT3
- net USB_DM renamed /mini-v1.14-macrofab-rtg_SS_1/USB_DM
- net USB_DP renamed /mini-v1.14-macrofab-rtg_SS_1/USB_DP
- net XSUM renamed /mini-v1.14-macrofab-rtg_SS_2/XSUM
- C1 pad 1: N$4 -> /mini-v1.14-macrofab-rtg_SS_1/N$4
- C15 pad 2: 6V -> /mini-v1.14-macrofab-rtg_SS_3/6V
- C17 pad P$1: VUSB -> 3V
- C18 pad P$1: VUSB -> 3V
- C19 pad P$1: VUSB -> 3V
- C20 pad P$1: VUSB -> 3V
- C3 pad P$1: 6V -> /mini-v1.14-macrofab-rtg_SS_3/6V
- C9 pad P$1: VUSB -> 3V
- D1 pad ANOD: (no net) -> 3V
- D1 pad CATH: (no net) -> /mini-v1.14-macrofab-rtg_SS_1/N$4
- L1 pad 1: VUSB -> 3V
- LD1 pad P$1: 6V -> /mini-v1.14-macrofab-rtg_SS_3/6V
- R17 pad P$2: 6V -> /mini-v1.14-macrofab-rtg_SS_3/6V
- R19 pad P$1: VUSB -> 3V
- R35 pad P$2: N$4 -> /mini-v1.14-macrofab-rtg_SS_1/N$4
- U$10 pad ANOD: (no net) -> GND
- U$10 pad CATH: (no net) -> 3V
- U$12 pad P5: VUSB -> 3V
- U$13 pad ANOD: (no net) -> GND
- U$13 pad CATH: (no net) -> 3V
- U$14 pad P$1: VUSB -> 3V
- U$14 pad P$2: N$15 -> /mini-v1.14-macrofab-rtg_SS_3/N$15
- U$15 pad 2: VUSB -> 3V
- U$16 pad 2: VUSB -> 3V
- U$17 pad 2: VUSB -> 3V
- U$5 pad 2: 6V -> /mini-v1.14-macrofab-rtg_SS_3/6V
- U$7 pad 2: VUSB -> 3V
- U$8 pad 1: N$15 -> /mini-v1.14-macrofab-rtg_SS_3/N$15
- U$8 pad 5: VUSB -> 3V
- U$9 pad ANOD: (no net) -> /mini-v1.14-macrofab-rtg_SS_3/N$15
- U$9 pad CATH: (no net) -> /mini-v1.14-macrofab-rtg_SS_3/6V
- U2 pad P$1: N$4 -> /mini-v1.14-macrofab-rtg_SS_1/N$4
- U2 pad P$3: N$4 -> /mini-v1.14-macrofab-rtg_SS_1/N$4
- VUSB71 pad TP: VUSB -> 3V
Routing:
- net 3V: track 155.8 -> 287.0 mm, vias 5 -> 10
- net VUSB: track 131.1 -> 0.00 mm, vias 5 -> 0
- net 6V: track 40.2 -> 0.00 mm
- net /mini-v1.14-macrofab-rtg_SS_3/6V: track 0.00 -> 40.2 mm
- net N$4: track 8.43 -> 0.00 mm
- net /mini-v1.14-macrofab-rtg_SS_1/N$4: track 0.00 -> 8.43 mm
- net N$15: track 7.12 -> 0.00 mm
- net /mini-v1.14-macrofab-rtg_SS_3/N$15: track 0.00 -> 7.12 mm
- net (no net): track 0.95 -> 0.00 mm, vias 1 -> 0
- net GND: track 137.1 -> 138.0 mm, vias 23 -> 24
